Commit message: positioning link0 and link1 on top of each other with joint

File: body.urdf (robot description, URDF)
Before this commit: robot robot, 2 links, 1 joints
Joints:
- joint link0_link1: origin xyz=0.5 0 1 rpy=0 0 0 -> xyz=0 0 1 rpy=0 0 0

Commit message: Added links 2-6 to create an archway

File: body.urdf (robot description, URDF)
Before this commit: robot robot, 2 links, 1 joints
Links:
- added link link2, mass 1; collision box size=1 1 1; visual box size=1 1 1
- added link link3, mass 1; collision box size=1 1 1; visual box size=1 1 1
- added link link4, mass 1; collision box size=1 1 1; visual box size=1 1 1
- added link link5, mass 1; collision box size=1 1 1; visual box size=1 1 1
- added link link6, mass 1; collision box size=1 1 1; visual box size=1 1 1
Joints:
- added joint link1_link2: type revolute, parent link1, child link2, origin xyz=0 0 1 rpy=0 0 0, axis 0 1 0, limit lower=-3.14159 upper=3.14159 effort=0.0 velocity=0.0
- added joint link2_link3: type revolute, parent link2, child link3, origin xyz=0.5 0 0.5 rpy=0 0 0, axis 0 1 0, limit lower=-3.14159 upper=3.14159 effort=0.0 velocity=0.0
- added joint link3_link4: type revolute, parent link3, child link4, origin xyz=1 0 0 rpy=0 0 0, axis 0 1 0, limit lower=-3.14159 upper=3.14159 effort=0.0 velocity=0.0
- added joint link4_link5: type revolute, parent link4, child link5, origin xyz=0.5 0 -0.5 rpy=0 0 0, axis 0 1 0, limit lower=-3.14159 upper=3.14159 effort=0.0 velocity=0.0
- added joint link5_link6: type revolute, parent link5, child link6, origin xyz=0 0 -1 rpy=0 0 0, axis 0 1 0, limit lower=-3.14159 upper=3.14159 effort=0.0 velocity=0.0

Commit message: Create torso, back and front legs

File: body.urdf (robot description, URDF)
Before this commit: robot robot, 7 links, 6 joints
Links:
- removed link link0
- removed link link1
- removed link link2
- removed link link3
- removed link link4
- removed link link5
- removed link link6
- added link backleg, mass 1; collision box size=1 1 1; visual box size=1 1 1
- added link frontleg, mass 1; collision box size=1 1 1; visual box size=1 1 1
- added link torso, mass 1; collision box size=1 1 1; visual box size=1 1 1
Joints:
- removed joint link0_link1
- removed joint link1_link2
- removed joint link2_link3
- removed joint link3_link4
- removed joint link4_link5
- removed joint link5_link6
- added joint torso_backleg: type revolute, parent torso, child backleg, origin xyz=-0.5 0 1 rpy=0 0 0, axis 0 1 0, limit lower=-3.14159 upper=3.14159 effort=0.0 velocity=0.0
- added joint torso_frontleg: type revolute, parent torso, child frontleg, origin xyz=0.5 0 1 rpy=0 0 0, axis 0 1 0, limit lower=-3.14159 upper=3.14159 effort=0.0 velocity=0.0

Commit message: Collisions_for_Donna

File: body.urdf (robot description, URDF)
Before this commit: robot robot, 3 links, 2 joints
Joints:
- joint torso_backleg: origin xyz=-0.5 0 1 rpy=0 0 0 -> xyz=1 0 1 rpy=0 0 0
- joint torso_frontleg: origin xyz=0.5 0 1 rpy=0 0 0 -> xyz=2 0 1 rpy=0 0 0

Commit message: added synapse to generate.py thru I.6

File: body.urdf (robot description, URDF)
Before this commit: robot robot, 3 links, 2 joints
Links:
- removed link backleg
- removed link frontleg
- removed link torso
- added link Backleg, mass 1; collision box size=1 1 1; visual box size=1 1 1
- added link Frontleg, mass 1; collision box size=1 1 1; visual box size=1 1 1
- added link Torso, mass 1; collision box size=1 1 1; visual box size=1 1 1
Joints:
- removed joint torso_backleg
- removed joint torso_frontleg
- added joint Torso_Backleg: type revolute, parent Torso, child Backleg, origin xyz=-0.5 0 1 rpy=0 0 0, axis 0 1 0, limit lower=-3.14159 upper=3.14159 effort=0.0 velocity=0.0
- added joint Torso_Frontleg: type revolute, parent Torso, child Frontleg, origin xyz=0.5 0 1 rpy=0 0 0, axis 0 1 0, limit lower=-3.14159 upper=3.14159 effort=0.0 velocity=0.0

Commit message: Thru M.18 - modify frontleg

File: body.urdf (robot description, URDF)
Before this commit: robot robot, 3 links, 2 joints
Links:
- link Frontleg: geometry collision box size=0.2 1 0.2; visual box size=0.2 1 0.2
Joints:
- joint Torso_Frontleg: origin xyz=0.5 0 1 rpy=0 0 0 -> xyz=0 0.5 1 rpy=0 0 0

Commit message: Thru N.22 - modify backleg

File: body.urdf (robot description, URDF)
Before this commit: robot robot, 3 links, 2 joints
Links:
- link Backleg: geometry collision box size=0.2 1 0.2; visual box size=0.2 1 0.2
Joints:
- joint Torso_Backleg: origin xyz=-0.5 0 1 rpy=0 0 0 -> xyz=0 -0.5 1 rpy=0 0 0

Commit message: Thru N.39 - adding left leg

File: body.urdf (robot description, URDF)
Before this commit: robot robot, 3 links, 2 joints
Links:
- added link Leftleg, mass 1; collision box size=1 0.2 0.2; visual box size=1 0.2 0.2
Joints:
- added joint Torso_Leftleg: type revolute, parent Torso, child Leftleg, origin xyz=-0.5 0 1 rpy=0 0 0, axis 0 1 0, limit lower=-3.14159 upper=3.14159 effort=0.0 velocity=0.0

Commit message: Thru N.40 - add right leg

File: body.urdf (robot description, URDF)
Before this commit: robot robot, 4 links, 3 joints
Links:
- added link Rightleg, mass 1; collision box size=1 0.2 0.2; visual box size=1 0.2 0.2
Joints:
- added joint Torso_Rightleg: type revolute, parent Torso, child Rightleg, origin xyz=0.5 0 1 rpy=0 0 0, axis 0 1 0, limit lower=-3.14159 upper=3.14159 effort=0.0 velocity=0.0

Commit message: thru N.42 - lower front leg

File: body.urdf (robot description, URDF)
Before this commit: robot robot, 5 links, 4 joints
Links:
- added link FrontLowerLeg, mass 1; collision box size=0.2 0.2 1; visual box size=0.2 0.2 1
Joints:
- added joint FrontLeg_FrontLowerLeg: type revolute, parent Frontleg, child FrontLowerLeg, origin xyz=0 1 0 rpy=0 0 0, axis 1 0 0, limit lower=-3.14159 upper=3.14159 effort=0.0 velocity=0.0

Commit message: Thru N.43 - added back lower leg

File: body.urdf (robot description, URDF)
Before this commit: robot robot, 6 links, 5 joints
Links:
- added link BackLowerLeg, mass 1; collision box size=0.2 0.2 1; visual box size=0.2 0.2 1
Joints:
- added joint BackLeg_BackLowerLeg: type revolute, parent Backleg, child BackLowerLeg, origin xyz=0 -1 0 rpy=0 0 0, axis 1 0 0, limit lower=-3.14159 upper=3.14159 effort=0.0 velocity=0.0

Commit message: Create lower left leg

File: body.urdf (robot description, URDF)
Before this commit: robot robot, 7 links, 6 joints
Links:
- added link LowerLeftLeg, mass 1; collision box size=0.2 0.2 1; visual box size=0.2 0.2 1
Joints:
- added joint LeftLeg_LowerLeftLeg: type revolute, parent Leftleg, child LowerLeftLeg, origin xyz=-1 0 0 rpy=0 0 0, axis 0 1 0, limit lower=-3.14159 upper=3.14159 effort=0.0 velocity=0.0

Commit message: Thru N.44 - added all lower legs

File: body.urdf (robot description, URDF)
Before this commit: robot robot, 8 links, 7 joints
Links:
- added link LowerRightLeg, mass 1; collision box size=0.2 0.2 1; visual box size=0.2 0.2 1
Joints:
- added joint RightLeg_LowerRightLeg: type revolute, parent Rightleg, child LowerRightLeg, origin xyz=1 0 0 rpy=0 0 0, axis 0 1 0, limit lower=-3.14159 upper=3.14159 effort=0.0 velocity=0.0

Commit message: All legs/joints have sensor and motor neurons

File: body.urdf (robot description, URDF)
Before this commit: robot robot, 9 links, 8 joints
Links:
- removed link LowerLeftLeg
- removed link LowerRightLeg
- added link LeftLowerLeg, mass 1; collision box size=0.2 0.2 1; visual box size=0.2 0.2 1
- added link RightLowerLeg, mass 1; collision box size=0.2 0.2 1; visual box size=0.2 0.2 1
Joints:
- removed joint LeftLeg_LowerLeftLeg
- removed joint RightLeg_LowerRightLeg
- added joint LeftLeg_LeftLowerLeg: type revolute, parent Leftleg, child LeftLowerLeg, origin xyz=-1 0 0 rpy=0 0 0, axis 0 1 0, limit lower=-3.14159 upper=3.14159 effort=0.0 velocity=0.0
- added joint RightLeg_RightLowerLeg: type revolute, parent Rightleg, child RightLowerLeg, origin xyz=1 0 0 rpy=0 0 0, axis 0 1 0, limit lower=-3.14159 upper=3.14159 effort=0.0 velocity=0.0

Commit message: First Attempt at Final Project

File: body.urdf (robot description, URDF)
Before this commit: robot robot, 9 links, 8 joints
Links:
- removed link BackLowerLeg
- removed link Backleg
- removed link FrontLowerLeg
- removed link Frontleg
- removed link LeftLowerLeg
- removed link Leftleg
- removed link RightLowerLeg
- removed link Rightleg
- removed link Torso
- added link Abdomen1, mass 1; collision box size=1 1 2; visual box size=1 1 2
- added link Abdomen2, mass 1; collision box size=1 1 2; visual box size=1 1 2
- added link Abdomen3, mass 1; collision box size=1 1 2; visual box size=1 1 2
- added link Head, mass 1; collision box size=1 1 2; visual box size=1 1 2
- added link Neck1, mass 1; collision box size=0.25 0.15 0.15; visual box size=0.25 0.15 0.15
- added link Neck2, mass 1; collision box size=0.25 0.15 0.15; visual box size=0.25 0.15 0.15
- added link Neck3, mass 1; collision box size=0.25 0.15 0.15; visual box size=0.25 0.15 0.15
Joints:
- removed joint BackLeg_BackLowerLeg
- removed joint FrontLeg_FrontLowerLeg
- removed joint LeftLeg_LeftLowerLeg
- removed joint RightLeg_RightLowerLeg
- removed joint Torso_Backleg
- removed joint Torso_Frontleg
- removed joint Torso_Leftleg
- removed joint Torso_Rightleg
- added joint Abdomen1_Neck2: type revolute, parent Abdomen1, child Neck2, origin xyz=1 0 0 rpy=0 0 0, axis 0 1 0, limit lower=-3.14159 upper=3.14159 effort=0.0 velocity=0.0
- added joint Abdomen2_Neck3: type revolute, parent Abdomen2, child Neck3, origin xyz=1 0 0 rpy=0 0 0, axis 0 1 0, limit lower=-3.14159 upper=3.14159 effort=0.0 velocity=0.0
- added joint Head_Neck1: type revolute, parent Head, child Neck1, origin xyz=0.5 0 1 rpy=0 0 0, axis 0 1 0, limit lower=-3.14159 upper=3.14159 effort=0.0 velocity=0.0
- added joint Neck1_Abdomen1: type revolute, parent Neck1, child Abdomen1, origin xyz=0.25 0 0 rpy=0 0 0, axis 0 1 0, limit lower=-3.14159 upper=3.14159 effort=0.0 velocity=0.0
- added joint Neck2_Abdomen2: type revolute, parent Neck2, child Abdomen2, origin xyz=0.25 0 0 rpy=0 0 0, axis 0 1 0, limit lower=-3.14159 upper=3.14159 effort=0.0 velocity=0.0
- added joint Neck3_Abdomen3: type revolute, parent Neck3, child Abdomen3, origin xyz=0.25 0 0 rpy=0 0 0, axis 0 1 0, limit lower=-3.14159 upper=3.14159 effort=0.0 velocity=0.0
